File: kicad/IotHenHouse.sch (KiCad schematic (older format))
At the start: 57 parts, among them J1 GND NC 5V RXD TXD NC, J2 Conn_01x02_Female, J3 3.3V SW1 SW2, M1 + MOT -, SW0 RESET, SW1 FLASH, U1 LM7805_TO220, U2 ESP-12E, U3 L298P, U4 LM1117-3.3

Commit message: mounting holes
Parts:
- added H1, H2, H3, H4: MountingHole, MountingHole:MountingHole_3.2mm_M3_Pad_Via, symbol Mechanical:MountingHole
- C1: footprint Capacitor_THT:CP_Radial_D22.0mm_P10.00mm_SnapIn -> Capacitor_THT:CP_Radial_D8.0mm_P2.50mm
Changed lines of the file:
@@
 F 0 "C1" H 2618 1546 50  0000 L CNN
 F 1 "330uF" H 2618 1455 50  0000 L CNN
-F 2 "Capacitor_THT:CP_Radial_D22.0mm_P10.00mm_SnapIn" H 2538 1350 50  0001 C CNN
+F 2 "Capacitor_THT:CP_Radial_D8.0mm_P2.50mm" H 2538 1350 50  0001 C CNN
 F 3 "~" H 2500 1500 50  0001 C CNN
 	1    2500 1500
@@
 Wire Wire Line
 	2000 1250 2500 1250
+$Comp
+L Mechanical:MountingHole H3
+U 1 1 608817C4
+P 9200 4950
+F 0 "H3" H 9300 4996 50  0000 L CNN
+F 1 "MountingHole" H 9300 4905 50  0000 L CNN
+F 2 "MountingHole:MountingHole_3.2mm_M3_Pad_Via" H 9200 4950 50  0001 C CNN
+F 3 "~" H 9200 4950 50  0001 C CNN
+	1    9200 4950
+	1    0    0    -1
+$EndComp
+$Comp
+L Mechanical:MountingHole H1
+U 1 1 60882202
+P 8450 4950
+F 0 "H1" H 8550 4996 50  0000 L CNN
+F 1 "MountingHole" H 8550 4905 50  0000 L CNN
+F 2 "MountingHole:MountingHole_3.2mm_M3_Pad_Via" H 8450 4950 50  0001 C CNN
+F 3 "~" H 8450 4950 50  0001 C CNN
+	1    8450 4950
+	1    0    0    -1
+$EndComp
+$Comp
+L Mechanical:MountingHole H4
+U 1 1 6088299C
+P 9200 5450
+F 0 "H4" H 9300 5496 50  0000 L CNN
+F 1 "MountingHole" H 9300 5405 50  0000 L CNN
+F 2 "MountingHole:MountingHole_3.2mm_M3_Pad_Via" H 9200 5450 50  0001 C CNN
+F 3 "~" H 9200 5450 50  0001 C CNN
+	1    9200 5450
+	1    0    0    -1
+$EndComp
+$Comp
+L Mechanical:MountingHole H2
+U 1 1 6088337D
+P 8450 5450
+F 0 "H2" H 8550 5496 50  0000 L CNN
+F 1 "MountingHole" H 8550 5405 50  0000 L CNN
+F 2 "MountingHole:MountingHole_3.2mm_M3_Pad_Via" H 8450 5450 50  0001 C CNN
+F 3 "~" H 8450 5450 50  0001 C CNN
+	1    8450 5450
+	1    0    0    -1
+$EndComp
 $EndSCHEMATC

Commit message: last commit for version 1.0
Connections:
- net +28V: no longer C9.1, U4.3 (VI)
- net +5V: now also C9.1, U4.3 (VI)
Changed lines of the file:
@@
 	1050 4100 1550 4100
-$Comp
-L power:+28V #PWR0104
-U 1 1 60471F3E
-P 1050 3800
-F 0 "#PWR0104" H 1050 3650 50  0001 C CNN
-F 1 "+28V" H 1065 3973 50  0000 C CNN
-F 2 "" H 1300 3850 50  0001 C CNN
-F 3 "" H 1300 3850 50  0001 C CNN
-	1    1050 3800
-	1    0    0    -1
-$EndComp
 $Comp
 L Device:LED D8
@@
 	1550 4150 1550 4100
 Connection ~ 1550 4100
-Connection ~ 1050 3800
 $Comp
 L power:+3.3V #PWR0107
@@
 	1    0    0    -1
 $EndComp
+$Comp
+L power:+5V #PWR0104
+U 1 1 610CFAA2
+P 1050 3750
+F 0 "#PWR0104" H 1050 3600 50  0001 C CNN
+F 1 "+5V" H 1065 3923 50  0000 C CNN
+F 2 "" H 1050 3750 50  0001 C CNN
+F 3 "" H 1050 3750 50  0001 C CNN
+	1    1050 3750
+	1    0    0    -1
+$EndComp
+Wire Wire Line
+	1050 3750 1050 3800
+Connection ~ 1050 3800
 $EndSCHEMATC
